File: DeeJ.kicad_pcb (KiCad board)
At the start: 2 copper layers, 303.9 x 187.3 mm, 129 parts, among them J1 USB_B_Micro, SW1 SW_Push, SW2 SW_DPDT_x2, SW3 SW_Push, SW5 SW_DPDT_x2, U1 DA04-11EWA, U3 MAX7219, U5 ESP32-S3-WROOM-1

Commit message: Small fixes
Parts:
- removed the D1 at (102.0, 169.5)
- removed the D1 at (120.5, 169.5)
- removed the RV2 at (120.5, 121.5)
- removed the RV2 at (83.5, 121.5)
- removed the RV2 at (102.0, 121.5)
- removed the SW3 at (120.5, 160.5)
- removed the SW3 at (102.0, 160.5)
- removed the U1 at (102.0, 86.0)
- removed the U1 at (120.5, 86.0)
- removed the U1 at (83.5, 86.0)
- added C1: 100nF, Capacitor_SMD:C_0805_2012Metric_Pad1.18x1.45mm_HandSolder, F.Cu at (-57.0, 112.9)
- added C1: 100nF, Capacitor_SMD:C_0805_2012Metric_Pad1.18x1.45mm_HandSolder, F.Cu at (-70.7, 112.9)
- added C1: 100nF, Capacitor_SMD:C_0805_2012Metric_Pad1.18x1.45mm_HandSolder, F.Cu at (-111.5, 112.9)
- added C1: 100nF, Capacitor_SMD:C_0805_2012Metric_Pad1.18x1.45mm_HandSolder, F.Cu at (59.5, 41.9)
- added C1: 100nF, Capacitor_SMD:C_0805_2012Metric_Pad1.18x1.45mm_HandSolder, F.Cu at (-125.0, 112.9)
- added C1: 100nF, Capacitor_SMD:C_0805_2012Metric_Pad1.18x1.45mm_HandSolder, F.Cu at (-84.2, 112.9)
- added C1: 100nF, Capacitor_SMD:C_0805_2012Metric_Pad1.18x1.45mm_HandSolder, F.Cu at (-97.8, 112.9)
- added C2: 100nF, Capacitor_SMD:C_0805_2012Metric_Pad1.18x1.45mm_HandSolder, F.Cu at (49.2, 39.3)
- added C2: 100nF, Capacitor_SMD:C_0805_2012Metric_Pad1.18x1.45mm_HandSolder, F.Cu at (-135.3, 110.3)
- added C2: 100nF, Capacitor_SMD:C_0805_2012Metric_Pad1.18x1.45mm_HandSolder, F.Cu at (-108.2, 110.3)
- added C2: 100nF, Capacitor_SMD:C_0805_2012Metric_Pad1.18x1.45mm_HandSolder, F.Cu at (-67.3, 110.3)
- added C2: 100nF, Capacitor_SMD:C_0805_2012Metric_Pad1.18x1.45mm_HandSolder, F.Cu at (-94.5, 110.3)
- added C2: 100nF, Capacitor_SMD:C_0805_2012Metric_Pad1.18x1.45mm_HandSolder, F.Cu at (-81.0, 110.3)
- added C2: 100nF, Capacitor_SMD:C_0805_2012Metric_Pad1.18x1.45mm_HandSolder, F.Cu at (-121.8, 110.3)
- added C3: 1uF, Capacitor_SMD:C_0805_2012Metric_Pad1.18x1.45mm_HandSolder, F.Cu at (-136.1, 39.3)
- added C4: 47uF, Capacitor_SMD:C_0805_2012Metric_Pad1.18x1.45mm_HandSolder, F.Cu at (-141.3, 45.3)
- added C5: 100nF, Capacitor_SMD:C_0805_2012Metric_Pad1.18x1.45mm_HandSolder, F.Cu at (-133.9, 39.3)
- added C6: 100nF, Capacitor_SMD:C_0805_2012Metric_Pad1.18x1.45mm_HandSolder, F.Cu at (-131.4, 176.0)
- added C6: 100nF, Capacitor_SMD:C_0805_2012Metric_Pad1.18x1.45mm_HandSolder, F.Cu at (-138.3, 48.4)
- added C7: 47nF, Capacitor_SMD:C_0805_2012Metric_Pad1.18x1.45mm_HandSolder, F.Cu at (-129.2, 176.0)
- added C7: 47nF, Capacitor_SMD:C_0805_2012Metric_Pad1.18x1.45mm_HandSolder, F.Cu at (-136.1, 48.4)
- added C8: 100nF, Capacitor_SMD:C_0805_2012Metric_Pad1.18x1.45mm_HandSolder, F.Cu at (19.5, 44.8)
- added C9: 1uF, Capacitor_SMD:C_0805_2012Metric_Pad1.18x1.45mm_HandSolder, F.Cu at (19.5, 47.8)
- added D1: LED, LED_THT:LED_D3.0mm, F.Cu at (204.0, 285.2)
- added D1: LED, LED_THT:LED_D3.0mm, F.Cu at (-299.1, 126.4)
- added D1: LED, LED_THT:LED_D3.0mm, F.Cu at (109.0, 168.5)
- added D1: LED, LED_THT:LED_D3.0mm, F.Cu at (191.8, 285.2)
- added D1: LED, LED_THT:LED_D3.0mm, F.Cu at (462.0, 384.5)
- added D1: LED, LED_THT:LED_D3.0mm, F.Cu at (122.0, 168.5)
- added D1: LED, LED_THT:LED_D3.0mm, F.Cu at (502.0, 384.5)
- added D1: LED, LED_THT:LED_D3.0mm, F.Cu at (218.0, 285.2)
- added D1: LED, LED_THT:LED_D3.0mm, F.Cu at (-325.1, 126.4)
- added D1: LED, LED_THT:LED_D3.0mm, F.Cu at (594.0, -22.8)
- added D1: LED, LED_THT:LED_D3.0mm, F.Cu at (502.0, 253.5)
- added D1: LED, LED_THT:LED_D3.0mm, F.Cu at (-312.1, 126.4)
- added D1: LED, LED_THT:LED_D3.0mm, F.Cu at (658.6, 137.9)
- added D1: LED, LED_THT:LED_D3.0mm, F.Cu at (167.5, 277.5)
- added D1: LED, LED_THT:LED_D3.0mm, F.Cu at (524.0, 253.5)
- added D1: LED, LED_THT:LED_D3.0mm, F.Cu at (135.0, 168.5)
- added D1: LED, LED_THT:LED_D3.0mm, F.Cu at (645.4, 137.9)
- added D1: LED, LED_THT:LED_D3.0mm, F.Cu at (710.6, 138.2)
- added D1: LED, LED_THT:LED_D3.0mm, F.Cu at (442.0, 253.5)
- added D1: LED, LED_THT:LED_D3.0mm, F.Cu at (482.0, 384.5)
- added D1: LED, LED_THT:LED_D3.0mm, F.Cu at (442.0, 384.5)
- added D1: LED, LED_THT:LED_D3.0mm, F.Cu at (482.0, 253.5)
- added D1: LED, LED_THT:LED_D3.0mm, F.Cu at (562.0, -22.8)
- added D1: LED, LED_THT:LED_D3.0mm, F.Cu at (529.0, -22.8)
- added D1: LED, LED_THT:LED_D3.0mm, F.Cu at (-364.1, 126.4)
- added D1: LED, LED_THT:LED_D3.0mm, F.Cu at (697.8, 137.9)
- added D1: LED, LED_THT:LED_D3.0mm, F.Cu at (546.0, -22.8)
- added D1: LED, LED_THT:LED_D3.0mm, F.Cu at (-351.1, 126.4)
- added D1: LED, LED_THT:LED_D3.0mm, F.Cu at (610.0, -22.8)
- added D1: LED, LED_THT:LED_D3.0mm, F.Cu at (26.9, 133.6)
- added D1: LED, LED_THT:LED_D3.0mm, F.Cu at (422.0, 253.5)
- added D1: LED, LED_THT:LED_D3.0mm, F.Cu at (179.5, 285.2)
- added D1: LED, LED_THT:LED_D3.0mm, F.Cu at (685.0, 137.9)
- added D1: LED, LED_THT:LED_D3.0mm, F.Cu at (578.0, -22.8)
- added D1: LED, LED_THT:LED_D3.0mm, F.Cu at (-338.1, 126.4)
- added D1: LED, LED_THT:LED_D3.0mm, F.Cu at (524.0, 384.5)
- added D1: LED, LED_THT:LED_D3.0mm, F.Cu at (671.6, 137.9)
- added D1: LED, LED_THT:LED_D3.0mm, F.Cu at (422.0, 384.5)
- added D1: LED, LED_THT:LED_D3.0mm, F.Cu at (148.0, 168.5)
- added D1: LED, LED_THT:LED_D3.0mm, F.Cu at (462.0, 253.5)
- added D1: LED, LED_THT:LED_D3.0mm, F.Cu at (161.0, 168.5)
- added D2: LED, LED_THT:LED_D3.0mm, F.Cu at (-76.1, 119.3)
- added D2: LED, LED_THT:LED_D3.0mm, F.Cu at (-123.0, 85.0)
- added D2: LED, LED_THT:LED_D3.0mm, F.Cu at (-103.6, 119.3)
- added D2: LED, LED_THT:LED_D3.0mm, F.Cu at (-117.3, 119.3)
- added D2: LED, LED_THT:LED_D3.0mm, F.Cu at (-90.0, 119.4)
- added D2: LED, LED_THT:LED_D3.0mm, F.Cu at (-131.0, 119.2)
- added D2: LED, LED_THT:LED_D3.0mm, F.Cu at (56.2, 43.2)
- added H2: MountingHole, MountingHole:M3spacer9mm, F.Cu at (515.8, 384.2)
- added H2: MountingHole, MountingHole:M3spacer9mm, F.Cu at (-140.4, 99.1)
- added H2: MountingHole, MountingHole:M3spacer9mm, F.Cu at (-52.0, 121.7)
- added H2: MountingHole, MountingHole:M3spacer9mm, F.Cu at (-140.0, 38.5)
- added H2: MountingHole, MountingHole:M3spacer9mm, F.Cu at (-52.0, 99.2)
- added H2: MountingHole, MountingHole:M3spacer9mm, F.Cu at (-140.1, 91.2)
- added H2: MountingHole, MountingHole:M3spacer9mm, F.Cu at (-140.4, 121.7)
- added H2: MountingHole, MountingHole:M3spacer9mm, F.Cu at (430.2, 384.2)
- added H2: MountingHole, MountingHole:M3spacer9mm, F.Cu at (-51.7, 68.8)
- added H2: MountingHole, MountingHole:M3spacer9mm, F.Cu at (-51.7, 91.3)
- added H2: MountingHole, MountingHole:M3spacer9mm, F.Cu at (-140.0, 61.1)
- added H2: MountingHole, MountingHole:M3spacer9mm, F.Cu at (-140.1, 68.7)
- added H2: MountingHole, MountingHole:M3spacer9mm, F.Cu at (-51.6, 61.1)
- added H2: MountingHole, MountingHole:M3spacer9mm, B.Cu at (104.6, -32.0)
- added H2: MountingHole, MountingHole:M3spacer9mm, F.Cu at (430.2, 315.8)
- added H2: MountingHole, MountingHole:M3spacer9mm, F.Cu at (515.8, 315.8)
- added H2: MountingHole, MountingHole:M3spacer9mm, F.Cu at (-51.6, 38.6)
- added J1: USB_C_Receptacle_USB2.0, Connector_USB:USB_C_Receptacle_HRO_TYPE-C-31-M-12, F.Cu at (452.0, 309.5)
- added J1: USB_C_Receptacle_USB2.0, Connector_USB:USB_C_Receptacle_HRO_TYPE-C-31-M-12, F.Cu at (452.0, 178.5)
- added J1: USB_C_Receptacle_USB2.0, Connector_USB:USB_C_Receptacle_HRO_TYPE-C-31-M-12, F.Cu at (-138.6, 196.1)
- added J1: USB_C_Receptacle_USB2.0, Connector_USB:USB_C_Receptacle_HRO_TYPE-C-31-M-12, F.Cu at (155.0, 274.0)
- added J2: Conn_02x08_Odd_Even, Connector_PinHeader_1.27mm:PinHeader_2x08_P1.27mm_Vertical, B.Cu at (-128.3, 68.0)
- added J3: Conn_02x08_Odd_Even, Connector_PinSocket_1.27mm:PinSocket_2x08_P1.27mm_Vertical, F.Cu at (663.6, 150.8)
- added J3: Conn_02x08_Odd_Even, Connector_PinSocket_1.27mm:PinSocket_2x08_P1.27mm_Vertical, F.Cu at (-115.5, 40.0)
- added J3: Conn_02x08_Odd_Even, Connector_PinSocket_1.27mm:PinSocket_2x08_P1.27mm_Vertical, B.Cu at (569.7, -55.3)
- added J3: Conn_02x08_Odd_Even, Connector_PinSocket_1.27mm:PinSocket_2x08_P1.27mm_Vertical, B.Cu at (569.7, -23.3)
- added R10: 10k, Resistor_SMD:R_0805_2012Metric_Pad1.20x1.40mm_HandSolder, F.Cu at (24.3, 47.7)
- added R2: 5k1, Resistor_SMD:R_0603_1608Metric_Pad0.98x0.95mm_HandSolder, F.Cu at (59.5, 44.0)
- added R2: 5k1, Resistor_SMD:R_0603_1608Metric_Pad0.98x0.95mm_HandSolder, F.Cu at (-70.7, 115.0)
- added R2: 5k1, Resistor_SMD:R_0603_1608Metric_Pad0.98x0.95mm_HandSolder, F.Cu at (-97.8, 115.0)
- added R2: 5k1, Resistor_SMD:R_0603_1608Metric_Pad0.98x0.95mm_HandSolder, F.Cu at (-57.0, 115.0)
- added R2: 5k1, Resistor_SMD:R_0603_1608Metric_Pad0.98x0.95mm_HandSolder, F.Cu at (-125.0, 115.0)
- added R2: 5k1, Resistor_SMD:R_0603_1608Metric_Pad0.98x0.95mm_HandSolder, F.Cu at (-84.2, 115.0)
- added R2: 5k1, Resistor_SMD:R_0603_1608Metric_Pad0.98x0.95mm_HandSolder, F.Cu at (-111.5, 115.0)
- added R3: 10k, Resistor_SMD:R_0805_2012Metric_Pad1.20x1.40mm_HandSolder, F.Cu at (-134.2, 114.9)
- added R3: 10k, Resistor_SMD:R_0805_2012Metric_Pad1.20x1.40mm_HandSolder, F.Cu at (-120.7, 114.9)
- added R3: 10k, Resistor_SMD:R_0805_2012Metric_Pad1.20x1.40mm_HandSolder, F.Cu at (-79.8, 114.9)
- added R3: 10k, Resistor_SMD:R_0805_2012Metric_Pad1.20x1.40mm_HandSolder, F.Cu at (-93.5, 114.9)
- added R3: 10k, Resistor_SMD:R_0805_2012Metric_Pad1.20x1.40mm_HandSolder, F.Cu at (50.3, 43.9)
- added R3: 10k, Resistor_SMD:R_0805_2012Metric_Pad1.20x1.40mm_HandSolder, F.Cu at (-107.0, 114.9)
- added R3: 10k, Resistor_SMD:R_0805_2012Metric_Pad1.20x1.40mm_HandSolder, F.Cu at (-66.2, 114.9)
- added R4: 10k, Resistor_SMD:R_0805_2012Metric_Pad1.20x1.40mm_HandSolder, F.Cu at (-79.8, 112.9)
- added R4: 10k, Resistor_SMD:R_0805_2012Metric_Pad1.20x1.40mm_HandSolder, F.Cu at (-107.0, 112.9)
- added R4: 10k, Resistor_SMD:R_0805_2012Metric_Pad1.20x1.40mm_HandSolder, F.Cu at (-134.2, 112.9)
- added R4: 10k, Resistor_SMD:R_0805_2012Metric_Pad1.20x1.40mm_HandSolder, F.Cu at (-66.2, 112.9)
- added R4: 10k, Resistor_SMD:R_0805_2012Metric_Pad1.20x1.40mm_HandSolder, F.Cu at (50.3, 41.9)
- added R4: 10k, Resistor_SMD:R_0805_2012Metric_Pad1.20x1.40mm_HandSolder, F.Cu at (-120.7, 112.9)
- added R4: 10k, Resistor_SMD:R_0805_2012Metric_Pad1.20x1.40mm_HandSolder, F.Cu at (-93.5, 112.9)
- added R5: R, Resistor_SMD:R_0805_2012Metric_Pad1.20x1.40mm_HandSolder, F.Cu at (-133.9, 48.4)
- added R5: R, Resistor_SMD:R_0805_2012Metric_Pad1.20x1.40mm_HandSolder, F.Cu at (-127.0, 176.0)
- added R6: 4k7, Resistor_SMD:R_0805_2012Metric_Pad1.20x1.40mm_HandSolder, F.Cu at (-140.5, 54.0)
- added R7: 220k, Resistor_SMD:R_0805_2012Metric_Pad1.20x1.40mm_HandSolder, F.Cu at (53.7, 165.0)
- added R8: 4k7, Resistor_SMD:R_0805_2012Metric_Pad1.20x1.40mm_HandSolder, F.Cu at (53.7, 159.6)
- added R9: 10k, Resistor_SMD:R_0805_2012Metric_Pad1.20x1.40mm_HandSolder, F.Cu at (24.3, 44.8)
- added REF**: ESP32-S3-WROOM-1U, Package_QFP:ESP32-S3-WROOM-1U, F.Cu at (114.2, -5.68)
- added REF**: LED_2512_6332Metric_Pad1.52x3.35mm_HandSolder, LED_SMD:LED_2512_6332Metric_Pad1.52x3.35mm_HandSolder, F.Cu at (33.0, 93.0)
- added REF**: 1551K, Enclosure:1551K, F.Cu at (417.0, 306.0)
- added REF**: PinHeader_2x10_P1.27mm_Vertical_SMD, Connector_PinHeader_1.27mm:PinHeader_2x10_P1.27mm_Vertical_SMD, F.Cu at (-58.7, 50.2)
- added REF**: LED_2512_6332Metric_Pad1.52x3.35mm_HandSolder, LED_SMD:LED_2512_6332Metric_Pad1.52x3.35mm_HandSolder, F.Cu at (37.5, 93.0)
- added REF**: PinSocket_2x10_P1.27mm_Vertical_SMD, Connector_PinSocket_1.27mm:PinSocket_2x10_P1.27mm_Vertical_SMD, B.Cu at (-59.1, 110.8)
- added REF**: ESP32-S3-WROOM-1U, Package_QFP:ESP32-S3-WROOM-1U, B.Cu at (114.7, 109.8)
- added REF**: ESP32-S3-WROOM-1U, Package_QFP:ESP32-S3-WROOM-1U, B.Cu at (230.2, 262.7)
- added REF**: 1551K, Enclosure:1551K, B.Cu at (227.0, 254.0)
- added REF**: QFN-56-1EP_7x7mm_P0.4mm_EP3.2x3.2mm, Package_DFN_QFN:QFN-56-1EP_7x7mm_P0.4mm_EP3.2x3.2mm, F.Cu at (-78.0, 49.1)
- added REF**: 1591XXABK, Enclosure:1591XXMBK, F.Cu at (522.6, -57.1)
- added REF**: ESP32-S3-WROOM-1U, Package_QFP:ESP32-S3-WROOM-1U, F.Cu at (-131.7, 182.9)
- added REF**: 1591XXMBK, Enclosure:1591XXMBK, F.Cu at (637.0, 102.8)
- added REF**: LED_2512_6332Metric_Pad1.52x3.35mm_HandSolder, LED_SMD:LED_2512_6332Metric_Pad1.52x3.35mm_HandSolder, F.Cu at (42.0, 93.0)
- added REF**: PinSocket_2x10_P1.27mm_Vertical_SMD, Connector_PinSocket_1.27mm:PinSocket_2x10_P1.27mm_Vertical_SMD, F.Cu at (-58.7, 50.2)
- added REF**: 1591XXGBK, Enclosure:1591XXGBK, F.Cu at (425.0, 306.0)
- added REF**: 1591XXGBK, Enclosure:1591XXGBK, F.Cu at (425.0, 175.0)
- added REF1**: Test point 2.5x1.5, TestPoint:Test point 2.5x1.5, F.Cu at (-0.40, 60.5)
- added RV1: R_Potentiometer, Potentiometer_THT:RS45111A900F, F.Cu at (-351.1, 78.9)
- added RV1: R_Potentiometer, Potentiometer_THT:RS45111A900F, F.Cu at (-364.1, 78.9)
- added RV1: R_Potentiometer, Potentiometer_THT:RS45111A900F, F.Cu at (161.0, 121.0)
- added RV1: R_Potentiometer, Potentiometer_THT:RS45111A900F, F.Cu at (502.0, 212.0)
- added RV1: R_Potentiometer, Potentiometer_THT:RS45111A900F, F.Cu at (148.0, 121.0)
- added RV1: R_Potentiometer, Potentiometer_THT:RS45111A900F, F.Cu at (-312.1, 78.9)
- added RV1: R_Potentiometer, Potentiometer_THT:RS45111A900F, F.Cu at (524.0, 343.0)
- added RV1: R_Potentiometer, Potentiometer_THT:RS45111A900F, F.Cu at (422.0, 343.0)
- added RV1: R_Potentiometer, Potentiometer_THT:RS45111A900F, F.Cu at (482.0, 343.0)
- added RV1: R_Potentiometer, Potentiometer_THT:RS45111A900F, F.Cu at (422.0, 212.0)
- added RV1: R_Potentiometer, Potentiometer_THT:RS45111A900F, F.Cu at (122.0, 121.0)
- added RV1: R_Potentiometer, Potentiometer_THT:RS45111A900F, F.Cu at (442.0, 343.0)
- added RV1: R_Potentiometer, Potentiometer_THT:RS45111A900F, F.Cu at (524.0, 212.0)
- added RV1: R_Potentiometer, Potentiometer_THT:RS45111A900F, F.Cu at (-338.1, 78.9)
- added RV1: R_Potentiometer, Potentiometer_THT:RS45111A900F, F.Cu at (135.0, 121.0)
- added RV1: R_Potentiometer, Potentiometer_THT:RS45111A900F, F.Cu at (-325.1, 78.9)
- added RV1: R_Potentiometer, Potentiometer_THT:RS45111A900F, F.Cu at (502.0, 343.0)
- added RV1: R_Potentiometer, Potentiometer_THT:RS45111A900F, F.Cu at (29.9, 118.5)
- added RV1: R_Potentiometer, Potentiometer_THT:RS45111A900F, F.Cu at (462.0, 343.0)
- added RV1: R_Potentiometer, Potentiometer_THT:RS45111A900F, F.Cu at (-299.1, 78.9)
- added RV1: R_Potentiometer, Potentiometer_THT:RS45111A900F, F.Cu at (109.0, 121.0)
- added RV1: R_Potentiometer, Potentiometer_THT:RS45111A900F, F.Cu at (482.0, 212.0)
- added RV1: R_Potentiometer, Potentiometer_THT:RS45111A900F, F.Cu at (442.0, 212.0)
- added RV1: R_Potentiometer, Potentiometer_THT:RS45111A900F, F.Cu at (462.0, 212.0)
- added RV3: R_Potentiometer, Potentiometer_THT:RK09K1130AST, F.Cu at (591.5, -35.2)
- added RV3: R_Potentiometer, Potentiometer_THT:RK09K1130AST, F.Cu at (-74.0, 175.0)
- added RV3: R_Potentiometer, Potentiometer_THT:RK09K1130AST, F.Cu at (680.9, 128.0)
- added RV3: R_Potentiometer, Potentiometer_THT:RK09K1130AST, F.Cu at (-126.8, 98.2)
- added RV3: R_Potentiometer, Potentiometer_THT:RK09K1130AST, F.Cu at (-73.1, 98.1)
- added RV3: R_Potentiometer, Potentiometer_THT:RK09K1130AST, F.Cu at (607.5, -35.2)
- added RV3: R_Potentiometer, Potentiometer_THT:RK09K1130AST, F.Cu at (-126.5, 82.0)
- added RV3: R_Potentiometer, Potentiometer_THT:RK09K1130AST, F.Cu at (-59.6, 98.1)
- added RV3: R_Potentiometer, Potentiometer_THT:RK09K1130AST, F.Cu at (543.5, -35.2)
- added RV3: R_Potentiometer, Potentiometer_THT:RK09K1130AST, F.Cu at (641.9, 128.0)
- added RV3: R_Potentiometer, Potentiometer_THT:RK09K1130AST, F.Cu at (559.5, -35.2)
- added RV3: R_Potentiometer, Potentiometer_THT:RK09K1130AST, F.Cu at (-86.5, 98.1)
- added RV3: R_Potentiometer, Potentiometer_THT:RK09K1130AST, F.Cu at (667.9, 128.0)
- added RV3: R_Potentiometer, Potentiometer_THT:RK09K1130AST, F.Cu at (706.9, 128.0)
- added RV3: R_Potentiometer, Potentiometer_THT:RK09K1130AST, F.Cu at (-60.0, 175.0)
- added RV3: R_Potentiometer, Potentiometer_THT:RK09K1130AST, F.Cu at (-102.0, 175.0)
- added RV3: R_Potentiometer, Potentiometer_THT:RK09K1130AST, F.Cu at (-46.0, 175.0)
- added RV3: R_Potentiometer, Potentiometer_THT:RK09K1130AST, F.Cu at (163.8, 267.3)
- added RV3: R_Potentiometer, Potentiometer_THT:RK09K1130AST, F.Cu at (188.2, 267.3)
- added RV3: R_Potentiometer, Potentiometer_THT:RK09K1130AST, F.Cu at (200.5, 267.3)
- added RV3: R_Potentiometer, Potentiometer_THT:RK09K1130AST, F.Cu at (693.9, 128.0)
- added RV3: R_Potentiometer, Potentiometer_THT:RK09K1130AST, F.Cu at (654.9, 128.0)
- added RV3: R_Potentiometer, Potentiometer_THT:RK09K1130AST, F.Cu at (176.0, 267.3)
- added RV3: R_Potentiometer, Potentiometer_THT:RK09K1130AST, F.Cu at (-100.0, 98.1)
- added RV3: R_Potentiometer, Potentiometer_THT:RK09K1130AST, F.Cu at (526.5, -35.2)
- added RV3: R_Potentiometer, Potentiometer_THT:RK09K1130AST, F.Cu at (-113.4, 98.1)
- added RV3: R_Potentiometer, Potentiometer_THT:RK09K1130AST, F.Cu at (575.5, -35.2)
- added RV3: R_Potentiometer, Potentiometer_THT:RK09K1130AST, F.Cu at (-88.0, 175.0)
- added RV4: R_Potentiometer, Potentiometer_SMD:Potentiometer_ACP_CA9-VSMD_Vertical, F.Cu at (52.4, 39.0)
- added RV5: R_Potentiometer, Potentiometer_THT:RK09K1130AST, F.Cu at (25.1, 74.0)
- added SW3: SW_Push, Button_Switch_THT:B3F-4055 with knob, F.Cu at (-364.1, 117.9)
- added SW3: SW_Push, Button_Switch_THT:B3F-4055 with knob, F.Cu at (-129.9, 113.9)
- added SW3: SW_Push, Button_Switch_THT:B3F-4055 with knob, F.Cu at (594.0, -29.3)
- added SW3: SW_Push, Button_Switch_THT:B3F-4055 with knob, F.Cu at (-299.1, 117.9)
- added SW3: SW_Push, Button_Switch_THT:B3F-4055 with knob, F.Cu at (562.0, -29.3)
- added SW3: SW_Push, Button_Switch_THT:B3F-4055 with knob, F.Cu at (-88.8, 114.1)
- added SW3: SW_Push, Button_Switch_THT:B3F-4055 with knob, F.Cu at (578.0, -29.3)
- added SW3: SW_Push, Button_Switch_THT:B3F-4055 with knob, F.Cu at (-351.1, 117.9)
- added SW3: SW_Push, Button_Switch_THT:B3F-4055 with knob, F.Cu at (109.0, 160.0)
- added SW3: SW_Push, Button_Switch_THT:B3F-4055 with knob, F.Cu at (122.0, 160.0)
- added SW3: SW_Push, Button_Switch_THT:B3F-4055 with knob, F.Cu at (-325.1, 117.9)
- added SW3: SW_Push, Button_Switch_THT:B3F-4055 with knob, F.Cu at (-75.0, 114.0)
- added SW3: SW_Push, Button_Switch_THT:B3F-4055 with knob, F.Cu at (148.0, 160.0)
- added SW3: SW_Push, Button_Switch_THT:B3F-4055 with knob, F.Cu at (-116.2, 114.0)
- added SW3: SW_Push, Button_Switch_THT:B3F-4055 with knob, F.Cu at (-338.1, 117.9)
- added SW3: SW_Push, Button_Switch_THT:B3F-4055 with knob, F.Cu at (135.0, 160.0)
- added SW3: SW_Push, Button_Switch_THT:B3F-4055 with knob, F.Cu at (161.0, 160.0)
- added SW3: SW_Push, Button_Switch_THT:B3F-4055 with knob, F.Cu at (529.0, -29.3)
- added SW3: SW_Push, Button_Switch_THT:B3F-4055 with knob, F.Cu at (546.0, -29.3)
- added SW3: SW_Push, Button_Switch_THT:B3F-4055 with knob, F.Cu at (-312.1, 117.9)
- added SW3: SW_Push, Button_Switch_THT:B3F-4055 with knob, F.Cu at (37.0, 135.0)
- added SW3: SW_Push, Button_Switch_THT:B3F-4055 with knob, F.Cu at (-102.5, 114.0)
- added SW4: SW_Push, Button_Switch_THT:SKHHCWA010, F.Cu at (594.0, -29.3)
- added SW4: SW_Push, Button_Switch_THT:SKHHCWA010, F.Cu at (696.5, 132.4)
- added SW4: SW_Push, Button_Switch_THT:SKHHCWA010, F.Cu at (462.0, 377.0)
- added SW4: SW_Push, Button_Switch_THT:SKHHCWA010, F.Cu at (422.0, 246.0)
- added SW4: SW_Push, Button_Switch_THT:SKHHCWA010, F.Cu at (-90.0, 191.0)
- added SW4: SW_Push, Button_Switch_THT:SKHHCWA010, F.Cu at (529.0, -29.3)
- added SW4: SW_Push, Button_Switch_THT:SKHHCWA010, F.Cu at (657.3, 132.4)
- added SW4: SW_Push, Button_Switch_THT:SKHHCWA010, F.Cu at (546.0, -29.3)
- added SW4: SW_Push, Button_Switch_THT:SKHHCWA010, F.Cu at (462.0, 246.0)
- added SW4: SW_Push, Button_Switch_THT:SKHHCWA010, F.Cu at (482.0, 377.0)
- added SW4: SW_Push, Button_Switch_THT:SKHHCWA010, F.Cu at (166.2, 272.0)
- added SW4: SW_Push, Button_Switch_THT:SKHHCWA010, F.Cu at (442.0, 377.0)
- added SW4: SW_Push, Button_Switch_THT:SKHHCWA010, F.Cu at (578.0, -29.3)
- added SW4: SW_Push, Button_Switch_THT:SKHHCWA010, F.Cu at (442.0, 246.0)
- added SW4: SW_Push, Button_Switch_THT:SKHHCWA010, F.Cu at (502.0, 246.0)
- added SW4: SW_Push, Button_Switch_THT:SKHHCWA010, F.Cu at (683.7, 132.4)
- added SW4: SW_Push, Button_Switch_THT:SKHHCWA010, F.Cu at (-48.0, 191.0)
- added SW4: SW_Push, Button_Switch_THT:SKHHCWA010, F.Cu at (54.9, 48.6)
- added SW4: SW_Push, Button_Switch_THT:SKHHCWA010, F.Cu at (670.3, 132.4)
- added SW4: SW_Push, Button_Switch_THT:SKHHCWA010, F.Cu at (-104.0, 191.0)
- added SW4: SW_Push, Button_Switch_THT:SKHHCWA010, F.Cu at (502.0, 377.0)
- added SW4: SW_Push, Button_Switch_THT:SKHHCWA010, F.Cu at (-76.0, 191.0)
- added SW4: SW_Push, Button_Switch_THT:SKHHCWA010, F.Cu at (482.0, 246.0)
- added SW4: SW_Push, Button_Switch_THT:SKHHCWA010, F.Cu at (709.3, 132.7)
- added SW4: SW_Push, Button_Switch_THT:SKHHCWA010, F.Cu at (524.0, 377.0)
- added SW4: SW_Push, Button_Switch_THT:SKHHCWA010, F.Cu at (-62.0, 191.0)
- added SW4: SW_Push, Button_Switch_THT:SKHHCWA010, F.Cu at (-124.0, 90.0)
- added SW4: SW_Push, Button_Switch_THT:SKHHCWA010, F.Cu at (562.0, -29.3)
- added SW4: SW_Push, Button_Switch_THT:SKHHCWA010, F.Cu at (610.0, -29.3)
- added SW4: SW_Push, Button_Switch_THT:SKHHCWA010, F.Cu at (524.0, 246.0)
- added SW4: SW_Push, Button_Switch_THT:SKHHCWA010, F.Cu at (422.0, 377.0)
- added SW4: SW_Push, Button_Switch_THT:SKHHCWA010, F.Cu at (644.1, 132.4)
- added SW6: SW_SPDT, Button_Switch_SMD:SK-3296S-01, F.Cu at (22.0, 39.9)
- added U1: USBLC6-2SC6, Package_TO_SOT_SMD:SOT-23-6, F.Cu at (-138.0, 178.0)
- added U2: 74HC14, Package_SO:TSSOP-14_4.4x5mm_P0.65mm, F.Cu at (202.1, 138.7)
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Connections:
- R1 pad 1: Net-(D1-K) -> Net-(J1-CC2) (x11)
- RV1 pad 1: (no net) -> unconnected-(RV1-Pad1) (x6)
- RV1 pad 2: (no net) -> unconnected-(RV1-Pad2) (x6)
- RV1 pad 3: (no net) -> unconnected-(RV1-Pad3) (x6)
- RV2 pad 1: (no net) -> unconnected-(RV2-Pad1)
- RV2 pad 2: (no net) -> unconnected-(RV2-Pad2)
- RV2 pad 3: (no net) -> unconnected-(RV2-Pad3)
- SW3 pad 1: (no net) -> unconnected-(SW3-Pad1) (x7)
- SW3 pad 2: (no net) -> unconnected-(SW3-Pad2) (x7)
- SW5 pad 1: unconnected-(SW5A-A-Pad1) -> Net-(C7-Pad1)
- SW5 pad 2: unconnected-(SW5A-B-Pad2) -> Net-(SW5-Pad2)
- U1 pad 1: (no net) -> Net-(J1-D--PadA7) (x7)
- U1 pad 2: (no net) -> GND (x7)
- U1 pad 3: (no net) -> Net-(J1-D+-PadA6) (x7)
- U1 pad 4: (no net) -> USB_D+ (x7)
- U1 pad 5: (no net) -> +5V (x7)
- U1 pad 6: (no net) -> USB_D- (x7)
- U3 pad 1: unconnected-(U3-DIN-Pad1) -> +3V3
- U3 pad 2: unconnected-(U3-DIG_0-Pad2) -> Net-(R3-Pad1)
- U3 pad 3: unconnected-(U3-DIG_4-Pad3) -> GND
- U3 pad 4: Net-(U3-GND-Pad4) -> GND
- U3 pad 1: (no net) -> +3V3
- U3 pad 2: (no net) -> Net-(R3-Pad1)
- U3 pad 3: (no net) -> GND
- U3 pad 4: (no net) -> GND
- U5 pad 1: unconnected-(U5-GND-Pad1) -> GND
- U5 pad 2: unconnected-(U5-3V3-Pad2) -> +3V3
- U5 pad 3: unconnected-(U5-EN-Pad3) -> +5V
Routing:
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- added copper zone on F.Cu, net +5V
- added copper zone on B.Cu, net GND
- added copper zone on F.Cu, net GND
Other:
- board size 303.9 x 187.3 mm -> 1095.9 x 451.1 mm
- board text added: "DWNLD"
- board text added: "OFF"
- board text added: "ON"
- board text added: "SPI BOOT"

Commit message: final design 1.0
Parts:
- removed the C1 at (-57.0, 112.9)
- removed the C1 at (-70.7, 112.9)
- removed the C1 at (-111.5, 112.9)
- removed the C1 at (59.5, 41.9)
- removed the C1 at (-125.0, 112.9)
- removed the C1 at (-84.2, 112.9)
- removed the C1 at (-97.8, 112.9)
- removed the C2 at (49.2, 39.3)
- removed the C2 at (-135.3, 110.3)
- removed the C2 at (-108.2, 110.3)
- removed the C2 at (-67.3, 110.3)
- removed the C2 at (-94.5, 110.3)
- removed the C2 at (-81.0, 110.3)
- removed the C2 at (-121.8, 110.3)
- removed the C6 at (-131.4, 176.0)
- removed the C6 at (-138.3, 48.4)
- removed the C7 at (-129.2, 176.0)
- removed the C7 at (-136.1, 48.4)
- removed D1 (x64), D2 (x7): LED, LED_THT:LED_D3.0mm
- removed H1 (x2), H2 (x23), H3 (x2), H4 (x2): MountingHole, MountingHole:M3spacer9mm
- removed the J1 at (452.0, 309.5)
- removed the J1 at (452.0, 178.5)
- removed the J1 at (-138.6, 196.1)
- removed the J1 at (155.0, 274.0)
- removed the J1 at (-146.5, 49.9)
- removed J2: Conn_02x08_Odd_Even, Connector_PinHeader_1.27mm:PinHeader_2x08_P1.27mm_Vertical
- removed J3 (x4): Conn_02x08_Odd_Even, Connector_PinSocket_1.27mm:PinSocket_2x08_P1.27mm_Vertical
- removed the R1 at (110.0, 44.0)
- removed the R1 at (79.5, 44.0)
- removed the R1 at (239.2, 122.0)
- removed the R1 at (255.2, 122.0)
- removed the R1 at (110.0, 61.0)
- removed the R1 at (225.1, 122.0)
- removed the R1 at (193.1, 122.0)
- removed the R1 at (140.0, 44.0)
- removed the R1 at (271.2, 122.0)
- removed the R1 at (209.1, 122.0)
- removed the R1 at (140.0, 61.0)
- removed R10, R9: 10k, Resistor_SMD:R_0805_2012Metric_Pad1.20x1.40mm_HandSolder
- removed the R2 at (59.5, 44.0)
- removed the R2 at (-70.7, 115.0)
- removed the R2 at (-97.8, 115.0)
- removed the R2 at (-57.0, 115.0)
- removed the R2 at (-125.0, 115.0)
- removed the R2 at (-84.2, 115.0)
- removed the R2 at (-111.5, 115.0)
- removed the R3 at (-134.2, 114.9)
- removed the R3 at (-120.7, 114.9)
- removed the R3 at (-79.8, 114.9)
- removed the R3 at (-93.5, 114.9)
- removed the R3 at (50.3, 43.9)
- removed the R3 at (-107.0, 114.9)
- removed the R3 at (-66.2, 114.9)
- removed the R4 at (-79.8, 112.9)
- removed the R4 at (-107.0, 112.9)
- removed the R4 at (-134.2, 112.9)
- removed the R4 at (-66.2, 112.9)
- removed the R4 at (50.3, 41.9)
- removed the R4 at (-120.7, 112.9)
- removed the R4 at (-93.5, 112.9)
- removed the R5 at (-133.9, 48.4)
- removed the R5 at (-127.0, 176.0)
- removed the REF** at (114.2, -5.68)
- removed the REF** at (33.0, 93.0)
- removed the REF** at (417.0, 306.0)
- removed the REF** at (-58.7, 50.2) (x2)
- removed the REF** at (37.5, 93.0)
- removed the REF** at (-59.1, 110.8)
- removed the REF** at (114.7, 109.8)
- removed the REF** at (230.2, 262.7)
- removed the REF** at (-0.30, 190.4)
- removed the REF** at (227.0, 254.0)
- removed the REF** at (-78.0, 49.1)
- removed the REF** at (522.6, -57.1)
- removed the REF** at (-131.7, 182.9)
- removed the REF** at (637.0, 102.8)
- removed the REF** at (42.0, 93.0)
- removed the REF** at (425.0, 306.0)
- removed the REF** at (425.0, 175.0)
- removed REF1**: Test point 2.5x1.5, TestPoint:Test point 2.5x1.5
- removed the RV1 at (317.1, 103.0)
- removed the RV1 at (-351.1, 78.9)
- removed the RV1 at (223.1, 107.0)
- removed the RV1 at (-364.1, 78.9)
- removed the RV1 at (208.9, 106.9)
- removed the RV1 at (269.2, 107.0)
- removed the RV1 at (161.0, 121.0)
- removed the RV1 at (317.1, 39.0)
- removed the RV1 at (502.0, 212.0)
- removed the RV1 at (148.0, 121.0)
- removed the RV1 at (-312.1, 78.9)
- removed the RV1 at (524.0, 343.0)
- removed the RV1 at (317.1, 87.0)
- removed the RV1 at (237.2, 107.0)
- removed the RV1 at (422.0, 343.0)
- removed the RV1 at (482.0, 343.0)
- removed the RV1 at (422.0, 212.0)
- removed the RV1 at (122.0, 121.0)
- removed the RV1 at (442.0, 343.0)
- removed the RV1 at (524.0, 212.0)
- removed the RV1 at (-338.1, 78.9)
- removed the RV1 at (135.0, 121.0)
- removed the RV1 at (-325.1, 78.9)
- removed the RV1 at (253.2, 107.0)
- removed the RV1 at (317.1, 55.0)
- removed the RV1 at (502.0, 343.0)
- removed the RV1 at (29.9, 118.5)
- removed the RV1 at (462.0, 343.0)
- removed the RV1 at (-299.1, 78.9)
- removed the RV1 at (96.0, 121.0)
- removed the RV1 at (317.1, 71.0)
- removed the RV1 at (109.0, 121.0)
- removed the RV1 at (482.0, 212.0)
- removed the RV1 at (442.0, 212.0)
- removed the RV1 at (462.0, 212.0)
- removed the RV1 at (317.1, 23.0)
- removed the RV2 at (351.0, 146.5)
- removed the RV2 at (218.0, 57.5)
- removed the RV2 at (312.0, 146.5)
- removed the RV2 at (338.0, 146.5)
- removed the RV2 at (344.0, 61.5)
- removed the RV2 at (325.0, 146.5)
- removed the RV2 at (299.0, 146.5)
- removed the RV2 at (364.0, 146.5)
- removed the RV2 at (208.0, 57.5)
- removed the RV2 at (198.0, 57.5)
- removed the RV2 at (188.0, 57.5)
- removed the RV2 at (178.0, 57.5)
- removed the RV3 at (591.5, -35.2)
- removed the RV3 at (-74.0, 175.0)
- removed the RV3 at (680.9, 128.0)
- removed the RV3 at (-126.8, 98.2)
- removed the RV3 at (-73.1, 98.1)
- removed the RV3 at (607.5, -35.2)
- removed the RV3 at (-126.5, 82.0)
- removed the RV3 at (-59.6, 98.1)
- removed the RV3 at (543.5, -35.2)
- removed the RV3 at (641.9, 128.0)
- removed the RV3 at (559.5, -35.2)
- removed the RV3 at (-86.5, 98.1)
- removed the RV3 at (667.9, 128.0)
- removed the RV3 at (124.5, 44.0)
- removed the RV3 at (706.9, 128.0)
- removed the RV3 at (-60.0, 175.0)
- removed the RV3 at (-102.0, 175.0)
- removed the RV3 at (-46.0, 175.0)
- removed the RV3 at (163.8, 267.3)
- removed the RV3 at (188.2, 267.3)
- removed the RV3 at (94.0, 44.0)
- removed the RV3 at (200.5, 267.3)
- removed the RV3 at (693.9, 128.0)
- removed the RV3 at (154.5, 61.0)
- removed the RV3 at (654.9, 128.0)
- removed the RV3 at (176.0, 267.3)
- removed the RV3 at (124.5, 61.0)
- removed the RV3 at (154.5, 44.0)
- removed the RV3 at (-100.0, 98.1)
- removed the RV3 at (526.5, -35.2)
- removed the RV3 at (-113.4, 98.1)
- removed the RV3 at (575.5, -35.2)
- removed the RV3 at (-88.0, 175.0)
- removed the SW1 at (218.0, 91.5)
- removed the SW1 at (208.0, 91.5)
- removed the SW1 at (218.1, 125.0)
- removed the SW1 at (178.0, 91.5)
- removed the SW1 at (186.1, 125.0)
- removed the SW1 at (248.2, 125.0)
- removed the SW1 at (232.2, 125.0)
- removed the SW1 at (202.1, 125.0)
- removed the SW1 at (188.0, 91.5)
- removed the SW1 at (198.0, 91.5)
- removed the SW1 at (264.2, 125.0)
- removed the SW2 at (83.5, 36.0)
- removed the SW2 at (144.0, 53.0)
- removed the SW2 at (114.0, 53.0)
- removed the SW2 at (114.0, 36.0)
- removed the SW2 at (144.0, 36.0)
- removed the SW3 at (96.0, 160.0)
- removed the SW3 at (-364.1, 117.9)
- removed the SW3 at (-129.9, 113.9)
- removed the SW3 at (351.0, 185.5)
- removed the SW3 at (594.0, -29.3)
- removed the SW3 at (-299.1, 117.9)
- removed the SW3 at (562.0, -29.3)
- removed the SW3 at (338.0, 185.5)
- removed the SW3 at (-88.8, 114.1)
- removed the SW3 at (578.0, -29.3)
- removed the SW3 at (297.5, 36.5)
- removed the SW3 at (-351.1, 117.9)
- removed the SW3 at (109.0, 160.0)
- removed the SW3 at (122.0, 160.0)
- removed the SW3 at (-325.1, 117.9)
- removed the SW3 at (-75.0, 114.0)
- removed the SW3 at (297.5, 84.5)
- removed the SW3 at (297.5, 68.5)
- removed the SW3 at (148.0, 160.0)
- removed the SW3 at (-116.2, 114.0)
- removed the SW3 at (299.0, 185.5)
- removed the SW3 at (610.0, -29.3)
- removed the SW3 at (-338.1, 117.9)
- removed the SW3 at (312.0, 185.5)
- removed the SW3 at (135.0, 160.0)
- removed the SW3 at (161.0, 160.0)
- removed the SW3 at (529.0, -29.3)
- removed the SW3 at (546.0, -29.3)
- removed the SW3 at (297.5, 100.5)
- removed the SW3 at (-312.1, 117.9)
- removed the SW3 at (297.5, 20.5)
- removed the SW3 at (37.0, 135.0)
- removed the SW3 at (-102.5, 114.0)
- removed the SW3 at (364.0, 185.5)
- removed the SW3 at (297.5, 52.5)
- removed the SW3 at (231.0, 78.5)
- removed the SW3 at (325.0, 185.5)
- removed the SW4 at (594.0, -29.3)
- removed the SW4 at (644.1, 132.4)
- removed the SW4 at (442.0, 377.0)
- removed the SW4 at (696.5, 132.4)
- removed the SW4 at (422.0, 246.0)
- removed the SW4 at (-90.0, 191.0)
- removed the SW4 at (529.0, -29.3)
- removed the SW4 at (657.3, 132.4)
- removed the SW4 at (546.0, -29.3)
- removed the SW4 at (462.0, 246.0)
- removed the SW4 at (166.2, 272.0)
- removed the SW4 at (524.0, 377.0)
- removed the SW4 at (578.0, -29.3)
- removed the SW4 at (442.0, 246.0)
- removed the SW4 at (502.0, 246.0)
- removed the SW4 at (683.7, 132.4)
- removed the SW4 at (-48.0, 191.0)
- removed the SW4 at (502.0, 377.0)
- removed the SW4 at (54.9, 48.6)
- removed the SW4 at (670.3, 132.4)
- removed the SW4 at (482.0, 377.0)
- removed the SW4 at (-104.0, 191.0)
- removed the SW4 at (482.0, 246.0)
- removed the SW4 at (-76.0, 191.0)
- removed the SW4 at (709.3, 132.7)
- removed the SW4 at (-62.0, 191.0)
- removed the SW4 at (-124.0, 90.0)
- removed the SW4 at (562.0, -29.3)
- removed the SW4 at (610.0, -29.3)
- removed the SW4 at (524.0, 246.0)
- removed the SW4 at (422.0, 377.0)
- removed the SW4 at (462.0, 377.0)
- removed the U1 at (-138.0, 178.0)
- removed the U1 at (326.0, 20.5)
- removed the U1 at (326.0, 68.5)
- removed the U1 at (344.0, 20.5)
- removed the U1 at (326.0, 52.5)
- removed the U1 at (326.0, 100.5)
- removed the U1 at (326.0, 36.5)
- removed the U1 at (326.0, 84.5)
- removed the U3 at (360.1, 22.5)
- removed the U3 at (363.6, 22.5)
- removed U5, U9 (x2): AMS1117-3.3, Package_TO_SOT_SMD:SOT-89-3_Handsoldering
- removed U6 (x3): ESP32-S3-WROOM-1, Package_QFP:ESP32-S3-WROOM-1
- removed U7: 74LVC2G14, Package_TO_SOT_SMD:SOT-363_SC-70-6_Handsoldering
- removed U8: ~, Button_Switch_SMD:SK-3296S-01
- added C1: 100nF, Capacitor_SMD:C_0805_2012Metric_Pad1.18x1.45mm_HandSolder, B.Cu at (155.0, 77.3)
- added C10: 100nF, Capacitor_SMD:C_0603_1608Metric_Pad1.08x0.95mm_HandSolder, F.Cu at (132.3, 71.9)
- added C11: 100nF, Capacitor_SMD:C_0603_1608Metric_Pad1.08x0.95mm_HandSolder, F.Cu at (132.3, 68.3)
- added C12: 1uF, Capacitor_SMD:C_0805_2012Metric_Pad1.18x1.45mm_HandSolder, F.Cu at (131.6, 99.8)
- added C13: 1uF, Capacitor_SMD:C_0805_2012Metric_Pad1.18x1.45mm_HandSolder, F.Cu at (124.8, 99.8)
- added C2: 100nF, Capacitor_SMD:C_0805_2012Metric_Pad1.18x1.45mm_HandSolder, B.Cu at (151.9, 84.5)
- added C6: 100nF, Capacitor_SMD:C_0603_1608Metric_Pad1.08x0.95mm_HandSolder, F.Cu at (148.1, 73.6)
- added C7: 100nF, Capacitor_SMD:C_0603_1608Metric_Pad1.08x0.95mm_HandSolder, F.Cu at (149.8, 73.6)
- added E1: ~, Enclosure:FIX-SF-664, B.Cu at (70.0, 45.0)
- added E2: ~, Enclosure:FIX-SF-664, B.Cu at (156.0, 45.0)
- added E3: ~, Enclosure:FIX-SF-664, B.Cu at (148.0, 111.0)
- added E4: ~, Enclosure:FIX-SF-664, B.Cu at (78.1, 111.0)
- added J1: USB_C_Receptacle_USB2.0, Connector_USB:USB_C_Receptacle_HRO_TYPE-C-31-M-12, F.Cu at (147.0, 38.0)
- added L1: 2.2uH, Inductor_SMD:L_TDK_VLS6045EX_VLS6045AF_handsolder, F.Cu at (129.4, 50.7)
- added Q1: SI2301S, Package_TO_SOT_SMD:SOT-23, B.Cu at (155.6, 97.1)
- added R1: 10k, Resistor_SMD:R_0805_2012Metric_Pad1.20x1.40mm_HandSolder, B.Cu at (154.0, 79.6)
- added R15: 100Ω, Resistor_SMD:R_0603_1608Metric_Pad0.98x0.95mm_HandSolder, F.Cu at (127.0, 111.0)
- added R16: 100Ω, Resistor_SMD:R_0603_1608Metric_Pad0.98x0.95mm_HandSolder, F.Cu at (144.0, 111.0)
- added R17: 100Ω, Resistor_SMD:R_0603_1608Metric_Pad0.98x0.95mm_HandSolder, F.Cu at (162.0, 111.0)
- added R18: 100Ω, Resistor_SMD:R_0603_1608Metric_Pad0.98x0.95mm_HandSolder, F.Cu at (110.0, 111.0)
- added R19: 100Ω, Resistor_SMD:R_0603_1608Metric_Pad0.98x0.95mm_HandSolder, F.Cu at (93.0, 111.0)
- added R2: 10k, Resistor_SMD:R_0805_2012Metric_Pad1.20x1.40mm_HandSolder, B.Cu at (139.6, 54.2)
- added R20: 100Ω, Resistor_SMD:R_0603_1608Metric_Pad0.98x0.95mm_HandSolder, F.Cu at (76.0, 111.0)
- added R3: 5k1, Resistor_SMD:R_0603_1608Metric_Pad0.98x0.95mm_HandSolder, B.Cu at (145.1, 38.2)
- added R4: 5k1, Resistor_SMD:R_0603_1608Metric_Pad0.98x0.95mm_HandSolder, B.Cu at (149.2, 38.2)
- added R5: 422k, Resistor_SMD:R_0603_1608Metric_Pad0.98x0.95mm_HandSolder, F.Cu at (128.1, 39.3)
- added REF**: 1551K, Enclosure:1551K, F.Cu at (62.0, 34.0)
- added RV1: R_Potentiometer, Potentiometer_THT:RS45111A900F, F.Cu at (121.0, 65.0)
- added RV2: R_Potentiometer, Potentiometer_THT:RS45111A900F, F.Cu at (138.0, 65.0)
- added RV3: R_Potentiometer, Potentiometer_THT:RS45111A900F, F.Cu at (156.0, 65.0)
- added RV6: R_Potentiometer, Potentiometer_THT:RS45111A900F, F.Cu at (70.0, 65.0)
- added SW1: SW_SPDT, Button_Switch_SMD:SK-3296S-01, B.Cu at (162.1, 51.8)
- added SW2: SW_SPDT, Button_Switch_SMD:SK-3296S-01, B.Cu at (162.1, 85.8)
- added SW3: SW_SPDT, Button_Switch_SMD:SK-3296S-01, B.Cu at (162.1, 98.6)
- added SW4: ~, Button_Switch_THT:K6-6133D, F.Cu at (121.0, 108.0)
- added SW7: ~, Button_Switch_THT:K6-6133D, F.Cu at (104.0, 108.0)
- added SW8: ~, Button_Switch_THT:K6-6133D, F.Cu at (87.0, 108.0)
- added SW9: ~, Button_Switch_THT:K6-6133D, F.Cu at (70.0, 108.0)
- added TP1: TestPoint, TestPoint:TestPoint_Pad_D2.0mm, F.Cu at (143.9, 50.4)
- added TP2: TestPoint, TestPoint:TestPoint_Pad_D2.0mm, F.Cu at (126.8, 60.4)
- added TP3: TestPoint, TestPoint:TestPoint_Pad_D2.0mm, F.Cu at (131.6, 94.6)
- added TP4: TestPoint, TestPoint:TestPoint_Pad_D2.0mm, F.Cu at (157.7, 96.9)
- added TP5: TestPoint, TestPoint:TestPoint_Pad_4.0x4.0mm, F.Cu at (112.4, 37.1)
- added U1: ESP32-S3-WROOM-1, Package_QFP:ESP32-S3-WROOM-1, B.Cu at (155.1, 74.8)
- added U3: TLV62569DBV, Package_TO_SOT_SMD:SOT-23-5, F.Cu at (128.9, 45.1)
- C3: moved to B.Cu
- C4: value 47uF -> 4.7uF; footprint Capacitor_SMD:C_0805_2012Metric_Pad1.18x1.45mm_HandSolder -> Capacitor_SMD:C_1206_3216Metric_Pad1.33x1.80mm_HandSolder
- C5: value 100nF -> 22uF
- C8: footprint Capacitor_SMD:C_0805_2012Metric_Pad1.18x1.45mm_HandSolder -> Capacitor_SMD:C_0603_1608Metric_Pad1.08x0.95mm_HandSolder
- C9: value 1uF -> 100nF; footprint Capacitor_SMD:C_0805_2012Metric_Pad1.18x1.45mm_HandSolder -> Capacitor_SMD:C_0603_1608Metric_Pad1.08x0.95mm_HandSolder
- R6: value 4k7 -> 100k; footprint Resistor_SMD:R_0805_2012Metric_Pad1.20x1.40mm_HandSolder -> Resistor_SMD:R_0603_1608Metric_Pad0.98x0.95mm_HandSolder
- R7: value 220k -> 10k; footprint Resistor_SMD:R_0805_2012Metric_Pad1.20x1.40mm_HandSolder -> Resistor_SMD:R_0603_1608Metric_Pad0.98x0.95mm_HandSolder; moved to B.Cu
- R8: value 4k7 -> 100Ω; footprint Resistor_SMD:R_0805_2012Metric_Pad1.20x1.40mm_HandSolder -> Resistor_SMD:R_0603_1608Metric_Pad0.98x0.95mm_HandSolder; moved to B.Cu
- RV4: footprint Potentiometer_SMD:Potentiometer_ACP_CA9-VSMD_Vertical -> Potentiometer_THT:RS45111A900F
- RV5: footprint Potentiometer_THT:RK09K1130AST -> Potentiometer_THT:RS45111A900F
- SW5: value SW_Push -> ~; footprint Button_Switch_THT:SKHHCWA010 -> Button_Switch_THT:K6-6133D
- SW6: value SW_SPDT -> ~; footprint Button_Switch_SMD:SK-3296S-01 -> Button_Switch_THT:K6-6133D
- U2: value 74HC14 -> USBLC6-2SC6; footprint Package_SO:TSSOP-14_4.4x5mm_P0.65mm -> Package_TO_SOT_SMD:SOT-23-6
- U4: footprint Button_Switch_SMD:SK-3296S-01 -> Package_TO_SOT_SMD:SOT-23-5
- moved C3 291.2 mm to (151.9, 82.2), turned to 180 degrees
- moved U4 280.7 mm to (128.2, 99.8), turned to 0 degrees
- moved C4 273.9 mm to (132.6, 44.5)
- moved R6 271.0 mm to (130.1, 39.3), turned to -90 degrees
- moved C5 262.2 mm to (127.8, 55.5), turned to 0 degrees
- moved SW6 150.3 mm to (156.0, 108.0), turned to 90 degrees
- moved C8 135.5 mm to (150.3, 80.2), turned to 180 degrees
- moved C9 129.5 mm to (146.4, 73.6), turned to 90 degrees
- moved R7 120.4 mm to (155.5, 100.7)
- moved R8 116.9 mm to (152.5, 97.1), turned to 90 degrees
- moved U2 106.7 mm to (147.0, 47.3), turned to -90 degrees
- moved SW5 94.5 mm to (138.0, 108.0), turned to 90 degrees
- moved RV5 62.5 mm to (87.0, 65.0), turned to 90 degrees
- moved RV4 57.8 mm to (104.0, 65.0)
Connections:
- C4 pad 1: +3V3 -> +5V
- C8 pad 1: EN -> /CH3
- C9 pad 1: EN -> /CH4
- R6 pad 1: Net-(C7-Pad1) -> GND
- R6 pad 2: MUTE_1 -> /SMPS_FB
- R7 pad 1: Net-(R7-Pad1) -> Net-(SW3-B)
- R7 pad 2: Net-(C7-Pad1) -> +3V3
- R8 pad 1: MUTE_1 -> Net-(SW3-B)
- RV4 pad 1: unconnected-(RV4-Pad1) -> Net-(SW7-1b)
- RV4 pad 2: unconnected-(RV4-Pad2) -> /CH4
- RV4 pad 3: unconnected-(RV4-Pad3) -> GND
- RV5 pad 1: GND -> Net-(SW8-1b)
- RV5 pad 2: VOL_1 -> /CH5
- RV5 pad 3: +3V3 -> GND
- SW5 pad 1: Net-(C7-Pad1) -> VDDA
- SW6 pad 1: +3V3 -> VDDA
- SW6 pad 4: GND -> Vled
- U2 pad 1: unconnected-(U2-Pad1) -> Net-(J1-D--PadA7)
- U2 pad 2: unconnected-(U2-Pad2) -> GND
- U2 pad 3: unconnected-(U2-Pad3) -> Net-(J1-D+-PadA6)
- U2 pad 4: unconnected-(U2-Pad4) -> USB_D+
- U2 pad 5: unconnected-(U2-Pad5) -> +5V
- U2 pad 6: unconnected-(U2-Pad6) -> USB_D-
- U4 pad 1: EN -> +5V
- U4 pad 3: GND -> +5V
- U4 pad 4: GND -> unconnected-(U4-NC-Pad4)
Routing:
- net Net-(J1-CC1): track 135.8 -> 3.86 mm, vias 14 -> 1
- net VDDA: track 0.00 -> 124.9 mm, vias 0 -> 2
- net Vled: track 0.00 -> 113.2 mm, vias 0 -> 1
- net (no net): track 112.3 -> 0.00 mm
- net unconnected-(SW4-Pad2): track 95.6 -> 0.00 mm
- net /CH6: track 0.00 -> 79.5 mm, vias 0 -> 1
- net /CH5: track 0.00 -> 61.0 mm, vias 0 -> 1
- net /CH4: track 0.00 -> 56.4 mm, vias 0 -> 1
- net +3V3: track 83.9 -> 130.2 mm, vias 2 -> 9
- net MUTE_1: track 43.6 -> 0.00 mm
- net /CH1: track 0.00 -> 40.4 mm, vias 0 -> 1
- net GND: track 32.2 -> 1.46 mm, vias 13 -> 40
- net Net-(D1-A): track 25.0 -> 0.00 mm
- net /CH2: track 0.00 -> 24.6 mm, vias 0 -> 1
- net USB_D-: track 5.77 -> 29.8 mm, vias 0 -> 1
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- added copper zone on F.Cu, net +3V3
- added copper zone on F.Cu, net /SMPS_SW
- removed copper zone on F.Cu, net +5V
Other:
- board size 1095.9 x 451.1 mm -> 102 x 82 mm
- board text added: "3V3"
- board text added: "5V"
- board text added: "GND"
- board text added: "VDDA"
- board text added: "VLED"
- board text removed: "DWNLD"
- board text removed: "OFF"
- board text removed: "ON"
- board text removed: "SPI BOOT"
