File: DeeJ.kicad_sch (KiCad schematic)
At the start: 18 parts, among them J1 USB_B_Micro, SW1 SW_Push, SW2 SW_DPDT_x2, SW3 SW_Push, SW5 SW_DPDT_x2, U1 DA04-11EWA, U3 MAX7219, U5 ESP32-S3-WROOM-1

Commit message: Small fixes
Parts:
- removed J1: USB_B_Micro, Connector_USB:USB_Micro-B_XKB_U254-051T-4BH83-F1S, symbol Connector:USB_B_Micro
- removed U1: DA04-11EWA, Display_7Segment:FJS-2281, symbol Display_Character:DA04-11EWA
- removed U2: ~, Display_7Segment:SP420281N, symbol Display_Character:SP420281N
- removed U3: MAX7219, Package_SO:SOIC-24W_7.5x15.4mm_P1.27mm, symbol Driver_LED:MAX7219
- added C1, C2, C5, C6, C8: 100nF, Capacitor_SMD:C_0805_2012Metric_Pad1.18x1.45mm_HandSolder, symbol Device:C
- added C3, C9: 1uF, Capacitor_SMD:C_0805_2012Metric_Pad1.18x1.45mm_HandSolder, symbol Device:C
- added C4: 47uF, Capacitor_SMD:C_0805_2012Metric_Pad1.18x1.45mm_HandSolder, symbol Device:C
- added C7: 47nF, Capacitor_SMD:C_0805_2012Metric_Pad1.18x1.45mm_HandSolder, symbol Device:C
- added D2: LED, LED_THT:LED_D3.0mm, symbol Device:LED
- added E1: ~, symbol Enclosure:1590B
- added J1: USB_C_Receptacle_USB2.0, Connector_USB:USB_C_Receptacle_HRO_TYPE-C-31-M-12, symbol Connector:USB_C_Receptacle_USB2.0
- added J2: Conn_02x08_Odd_Even, Connector_PinHeader_1.27mm:PinHeader_2x08_P1.27mm_Vertical, symbol Connector_Generic:Conn_02x08_Odd_Even
- added J3: Conn_02x08_Odd_Even, Connector_PinSocket_1.27mm:PinSocket_2x08_P1.27mm_Vertical, symbol Connector_Generic:Conn_02x08_Odd_Even
- added R1, R2: 5k1, Resistor_SMD:R_0603_1608Metric_Pad0.98x0.95mm_HandSolder, symbol Device:R
- added R10, R3, R4, R9: 10k, Resistor_SMD:R_0805_2012Metric_Pad1.20x1.40mm_HandSolder, symbol Device:R
- added R6, R8: 4k7, Resistor_SMD:R_0805_2012Metric_Pad1.20x1.40mm_HandSolder, symbol Device:R
- added R7: 220k, Resistor_SMD:R_0805_2012Metric_Pad1.20x1.40mm_HandSolder, symbol Device:R
- added RV4: R_Potentiometer, Potentiometer_SMD:Potentiometer_ACP_CA9-VSMD_Vertical, symbol Device:R_Potentiometer
- added RV5: R_Potentiometer, Potentiometer_THT:RK09K1130AST, symbol Device:R_Potentiometer
- added SW5: SW_Push, Button_Switch_THT:SKHHCWA010, symbol Switch:SW_Push
- added SW6: SW_SPDT, Button_Switch_SMD:SK-3296S-01, symbol Switch:SW_SPDT_shielded
- added SW7: SW_SPDT, symbol Switch:SW_SPDT_shielded
- added U1: USBLC6-2SC6, Package_TO_SOT_SMD:SOT-23-6, symbol Power_Protection:USBLC6-2SC6
- added U2: 74HC14, Package_SO:TSSOP-14_4.4x5mm_P0.65mm, symbol 74xx:74HC14
- added U3, U4: ~, Button_Switch_SMD:SK-3296S-01, symbol Switch:SPDT_grounded
- added U5: AMS1117-3.3, Package_TO_SOT_SMD:SOT-89-3_Handsoldering, symbol Regulator_Linear:AMS1117-3.3
- added U7: 74LVC2G14, Package_TO_SOT_SMD:SOT-363_SC-70-6_Handsoldering, symbol 74xGxx:74LVC2G14_1
- renumbered R1 to R5, RV2 to RV1, RV3 to RV2, RV1 to RV3, SW5 to SW1, SW1 to SW4, U5 to U6
Connections:
- net +3V3: now also U6.2 (3V3), C4.1, C5.1, C6.1, R10.2, R4.2, RV5.3, SW6.1 (A), U3.1, U5.2 (VO), U7.5 (VCC)
- net GND: now also U6.1 (GND), U6.40 (GND), U6.41 (GND), C1.2, C2.2, C3.2, C4.2, C5.2, C6.2, C7.2, C8.2, C9.2, D2.1 (K), J1.A1 (GND), J1.A12 (GND), J1.B1 (GND), J1.B12 (GND), J1.S1 (SHIELD), R1.2, R2.2, RV5.1, SW6.3 (C), SW6.4 (Shield), SW7.2 (B), SW7.3 (C), SW7.4 (Shield), U1.2 (GND), U3.3, U3.4 (GND), U4.2, U4.3, U4.4 (GND), U5.1 (GND), U7.2 (GND)
- net USB_D-: now reaches U6.13 (IO19)
- net USB_D-: now also U1.6 (I/O2)
- net USB_D+: now reaches U6.14 (IO20)
- net USB_D+: now also U1.4 (I/O2)
- net MUTE_4: now reaches U6.22 (1014)
- net MUTE_3: now reaches U6.23 (IO21)
- net MUTE_2: now reaches U6.24 (IO47)
- net MUTE_1: now reaches U6.25 (IO48)
- net MUTE_1: now also R6.2, R8.1, U7.4
- net BOOT: now reaches U6.27 (IO0)
- net BOOT: now also R3.2, R9.2
- net EN: now reaches U6.3 (EN)
- net EN: now also C1.1, C3.1, C8.1, C9.1, R10.1, R4.1, SW7.1 (A), U4.1
- net MUTE_5: now reaches U6.31 (IO38)
- net TCK: now reaches U6.32 (IO39)
- net TDO: now reaches U6.33 (IO40)
- net TDI: now reaches U6.34 (IO41)
- net TMS: now reaches U6.35 (IO42)
- net VOL_1: now reaches U6.4 (IO4)
- net VOL_1: now also RV5.2
- net VOL_2: now reaches U6.5 (IO5)
- net VOL_3: now reaches U6.6 (IO6)
- net VOL_4: now reaches U6.7 (IO7)
- net VOL_5: now reaches U6.8 (IO15)
- new net: J1.A7 (D-), J1.B7 (D-), U1.1 (I/O1)
- new net: J1.A6 (D+), J1.B6 (D+), U1.3 (I/O1)
- new net: R9.1, SW6.2 (B)
- new net: C7.1, R6.1, R7.2, SW5.1
- new net: J1.B5 (CC2), R1.1
- new net: R7.1, U7.3, U7.6
- new net: J1.A5 (CC1), R2.1
- new net: R3.1, U3.2
- new net: SW5.2, U7.1
- new net: D2.2 (A), R8.2
- new net +5V: C2.1, J1.A4 (VBUS), J1.A9 (VBUS), J1.B4 (VBUS), J1.B9 (VBUS), U1.5 (VBUS), U5.3 (VI)
- no-connect marks 0 -> 2
Other:
- note added: "1591XXABK"
- note added: "C2935886"
- note added: "C2935956"
- note added: "ESP32 BOOT AND ENABLE"
- note added: "Kotelo ehdokas 1591XXGSBK"
- note added: "USB with ESD protection and CC pulldowns"
- note added: "Usb C to A cable C430908"
- note added: "iso liukuboxi"
- note added: "pcb interconnect spacing 5mm"
- note added: "pisla kumitassu 100x150mm 4.19€"
- note added: "potentiometer to panel heights slide = 7mm rotary = 7mm"
- note added: "ruuvi C357483 1.7x5 C357489 2.3x5 C357380 2x5 C5222489 3x5"
- moved on the sheet: H1, H2, H3, H4, RV2, SW4

Commit message: final design 1.0
Parts:
- removed C1, C2, C6: 100nF, Capacitor_SMD:C_0805_2012Metric_Pad1.18x1.45mm_HandSolder, symbol Device:C
- removed C3: 1uF, Capacitor_SMD:C_0805_2012Metric_Pad1.18x1.45mm_HandSolder, symbol Device:C
- removed C7: 47nF, Capacitor_SMD:C_0805_2012Metric_Pad1.18x1.45mm_HandSolder, symbol Device:C
- removed D1, D2: LED, LED_THT:LED_D3.0mm, symbol Device:LED
- removed H1, H2, H3, H4: MountingHole, MountingHole:M3spacer9mm, symbol Mechanical:MountingHole
- removed J2: Conn_02x08_Odd_Even, Connector_PinHeader_1.27mm:PinHeader_2x08_P1.27mm_Vertical, symbol Connector_Generic:Conn_02x08_Odd_Even
- removed J3: Conn_02x08_Odd_Even, Connector_PinSocket_1.27mm:PinSocket_2x08_P1.27mm_Vertical, symbol Connector_Generic:Conn_02x08_Odd_Even
- removed R3, R4: 10k, Resistor_SMD:R_0805_2012Metric_Pad1.20x1.40mm_HandSolder, symbol Device:R
- removed RV1: R_Potentiometer, Potentiometer_THT:RS45111A900F, symbol Device:R_Potentiometer
- removed RV2: R_Potentiometer, Potentiometer_THT:RK09D1130C2P, symbol Device:R_Potentiometer
- removed RV3, RV5: R_Potentiometer, Potentiometer_THT:RK09K1130AST, symbol Device:R_Potentiometer
- removed RV4: R_Potentiometer, Potentiometer_SMD:Potentiometer_ACP_CA9-VSMD_Vertical, symbol Device:R_Potentiometer
- removed SW1: SW_DPDT_x2, Button_Switch_THT:SPEF110100, symbol Switch:SW_DPDT_x2
- removed SW2: SW_DPDT_x2, Button_Switch_THT:SPPH110900, symbol Switch:SW_DPDT_x2
- removed SW3: SW_Push, Button_Switch_THT:B3F-4055 with knob, symbol Switch:SW_Push
- removed SW4, SW5: SW_Push, Button_Switch_THT:SKHHCWA010, symbol Switch:SW_Push
- removed U2: 74HC14, Package_SO:TSSOP-14_4.4x5mm_P0.65mm, symbol 74xx:74HC14
- removed U3, U4: ~, Button_Switch_SMD:SK-3296S-01, symbol Switch:SPDT_grounded
- removed U5: AMS1117-3.3, Package_TO_SOT_SMD:SOT-89-3_Handsoldering, symbol Regulator_Linear:AMS1117-3.3
- removed U7: 74LVC2G14, Package_TO_SOT_SMD:SOT-363_SC-70-6_Handsoldering, symbol 74xGxx:74LVC2G14_1
- added C12, C13: 1uF, Capacitor_SMD:C_0805_2012Metric_Pad1.18x1.45mm_HandSolder, symbol Device:C
- added C5: 22uF, Capacitor_SMD:C_0805_2012Metric_Pad1.18x1.45mm_HandSolder, symbol Device:C
- added E2, E3, E4: ~, Enclosure:FIX-SF-664, symbol Enclosure:1590B
- added L1: 2.2uH, Inductor_SMD:L_TDK_VLS6045EX_VLS6045AF_handsolder, symbol Device:L
- added Q1: SI2301S, Package_TO_SOT_SMD:SOT-23, symbol Simulation_SPICE:PMOS
- added SW3: SW_SPDT, Button_Switch_SMD:SK-3296S-01, symbol Switch:SW_SPDT_shielded
- added TP1, TP2, TP3, TP4: TestPoint, TestPoint:TestPoint_Pad_D2.0mm, symbol Connector:TestPoint
- added TP5: TestPoint, TestPoint:TestPoint_Pad_4.0x4.0mm, symbol Connector:TestPoint
- added U3: TLV62569DBV, Package_TO_SOT_SMD:SOT-23-5, symbol Regulator_Switching:TLV62569DBV
- added U4: ~, Package_TO_SOT_SMD:SOT-23-5, symbol Regulator_Linear:TPS7A20
- C4: value 47uF -> 4.7uF; footprint Capacitor_SMD:C_0805_2012Metric_Pad1.18x1.45mm_HandSolder -> Capacitor_SMD:C_1206_3216Metric_Pad1.33x1.80mm_HandSolder; ESR (none) -> 3.417mΩ; LCSC# (none) -> C527983
- E1: footprint (none) -> Enclosure:FIX-SF-664
- R5: value R -> 422k; footprint Resistor_SMD:R_0805_2012Metric_Pad1.20x1.40mm_HandSolder -> Resistor_SMD:R_0603_1608Metric_Pad0.98x0.95mm_HandSolder; Power (none) -> 1/16W; Tolerance (none) -> 1%
- R6: value 4k7 -> 100k; footprint Resistor_SMD:R_0805_2012Metric_Pad1.20x1.40mm_HandSolder -> Resistor_SMD:R_0603_1608Metric_Pad0.98x0.95mm_HandSolder; Power (none) -> 1/16W; Tolerance (none) -> 1%
- R7: value 220k -> 10k; footprint Resistor_SMD:R_0805_2012Metric_Pad1.20x1.40mm_HandSolder -> Resistor_SMD:R_0603_1608Metric_Pad0.98x0.95mm_HandSolder
- R8: value 4k7 -> 100Ω; footprint Resistor_SMD:R_0805_2012Metric_Pad1.20x1.40mm_HandSolder -> Resistor_SMD:R_0603_1608Metric_Pad0.98x0.95mm_HandSolder
- SW2: renamed from SW7; footprint (none) -> Button_Switch_SMD:SK-3296S-01
- renumbered C5 to C1, C8 to C2, C9 to C3, R10 to R1, R9 to R2, R1 to R3, R2 to R4, SW6 to SW1, U6 to U1, U1 to U2
Connections:
- net +3V3: now also R5.2, R7.2, C5.1, L1.2, Q1.3 (S), SW3.1 (A), TP2.1; no longer C4.1
- net +5V: now also C4.1, C13.1, TP1.1, U3.1 (EN), U3.4 (VIN), U4.1 (Vin), U4.3 (EN)
- net GND: now also R6.1, C12.2, C13.2, C5.2, SW3.3 (C), SW3.4 (Shield), TP5.1, U3.2 (GND), U4.2 (GND); no longer R5.2
- net at R7.1: now also R8.1, SW3.2 (B)
- net at R8.2: now also Q1.2 (G)
- net CH5: now reaches U1.17 (IO9)
- net CH6: now reaches U1.18 (IO10)
- net SMPS_FB: now reaches R5.1
- net SMPS_FB: now also R6.2, U3.5 (FB)
- removed net MUTE_1: R6.2, R8.1, U1.25 (IO48)
- net MUTE_2: no longer names the net of U1.24 (IO47)
- net MUTE_3: no longer names the net of U1.23 (IO21)
- net MUTE_4: no longer names the net of U1.22 (1014)
- net MUTE_5: no longer names the net of U1.31 (IO38)
- net VOL_1 renamed CH3
- net VOL_2 renamed CH2
- net VOL_3 renamed CH1
- net VOL_4 renamed CH4
- net VOL_5: no longer names the net of U1.8 (IO15)
- new net SMPS_SW: L1.1, U3.3 (SW)
- new net VDDA: C12.1, TP3.1, U4.5 (Vout)
- new net Vled: Q1.1 (D), TP4.1
Other:
- added sheet CH1 (CH.kicad_sch)
- added sheet CH2 (CH.kicad_sch)
- added sheet CH3 (CH.kicad_sch)
- added sheet CH4 (CH.kicad_sch)
- added sheet CH5 (CH.kicad_sch)
- added sheet CH6 (CH.kicad_sch)
- note added: "5V to 3V3 buck converter"
- note added: "LED switch"
- note added: "Precission analog supply"
- moved on the sheet: C1, C2, C3, J1, R1, R2, R3, R4, SW1, SW2, U1, U2
